File: west_workshop_2025.kicad_pcb (KiCad board)
At the start: 4 copper layers, 0 parts

Commit message: Clean PCB.
Other:
- copper layers 4 -> 2

Commit message: Finished PCB
Parts:
- added A1: RaspberryPi_Pico, 0_west_footprints:RaspberryPi_Pico, B.Cu at (155.3, 72.0)
- added D1: LED, 0_west_footprints:Kingbright_WP914x, F.Cu at (121.0, 82.3)
- added D10: 1N4148, Diode_THT:D_DO-35_SOD27_P7.62mm_Horizontal, F.Cu at (121.0, 126.0)
- added D11: 1N4148, Diode_THT:D_DO-35_SOD27_P7.62mm_Horizontal, F.Cu at (126.8, 126.0)
- added D12: 1N4148, Diode_THT:D_DO-35_SOD27_P7.62mm_Horizontal, F.Cu at (132.6, 126.0)
- added D13: 1N4148, Diode_THT:D_DO-35_SOD27_P7.62mm_Horizontal, F.Cu at (138.4, 126.0)
- added D14: 1N4148, Diode_THT:D_DO-35_SOD27_P7.62mm_Horizontal, F.Cu at (144.2, 126.0)
- added D15: 1N4148, Diode_THT:D_DO-35_SOD27_P7.62mm_Horizontal, F.Cu at (150.1, 126.0)
- added D16: 1N4148, Diode_THT:D_DO-35_SOD27_P7.62mm_Horizontal, F.Cu at (155.9, 126.0)
- added D17: 1N4148, Diode_THT:D_DO-35_SOD27_P7.62mm_Horizontal, F.Cu at (161.7, 126.0)
- added D18: 1N4148, Diode_THT:D_DO-35_SOD27_P7.62mm_Horizontal, F.Cu at (167.5, 125.9)
- added D2: LED, 0_west_footprints:Kingbright_WP914x, F.Cu at (140.0, 82.3)
- added D3: LED, 0_west_footprints:Kingbright_WP914x, F.Cu at (159.1, 82.3)
- added D4: LED, 0_west_footprints:Kingbright_WP914x, F.Cu at (121.0, 101.4)
- added D5: LED, 0_west_footprints:Kingbright_WP914x, F.Cu at (140.0, 101.4)
- added D6: LED, 0_west_footprints:Kingbright_WP914x, F.Cu at (159.1, 101.4)
- added D7: LED, 0_west_footprints:Kingbright_WP914x, F.Cu at (121.0, 120.4)
- added D8: LED, 0_west_footprints:Kingbright_WP914x, F.Cu at (140.0, 120.4)
- added D9: LED, 0_west_footprints:Kingbright_WP914x, F.Cu at (159.1, 120.4)
- added G***: LOGO, 0_west_footprints:SELogo, F.Cu at (127.8, 62.8)
- added G***: LOGO, 0_west_footprints:WESTLogo, B.Cu at (165.5, 64.0)
- added H1: MountingHole, 0_west_footprints:MountingHole_M2, F.Cu at (115.0, 62.2)
- added H2: MountingHole, 0_west_footprints:MountingHole_M2, F.Cu at (177.8, 62.2)
- added H3: MountingHole, 0_west_footprints:MountingHole_M2, F.Cu at (115.0, 135.0)
- added H4: MountingHole, 0_west_footprints:MountingHole_M2, F.Cu at (177.8, 135.0)
- added Q1: TN0604, Package_TO_SOT_THT:TO-92L_Inline, F.Cu at (172.2, 128.1)
- added R1: 390R, Resistor_THT:R_Axial_DIN0204_L3.6mm_D1.6mm_P5.08mm_Horizontal, B.Cu at (116.0, 67.9)
- added R10: 390R, Resistor_THT:R_Axial_DIN0204_L3.6mm_D1.6mm_P5.08mm_Horizontal, B.Cu at (177.0, 105.3)
- added R11: 10k, Resistor_THT:R_Axial_DIN0204_L3.6mm_D1.6mm_P5.08mm_Horizontal, B.Cu at (177.0, 119.8)
- added R2: 390R, Resistor_THT:R_Axial_DIN0204_L3.6mm_D1.6mm_P5.08mm_Horizontal, B.Cu at (116.0, 77.3)
- added R3: 390R, Resistor_THT:R_Axial_DIN0204_L3.6mm_D1.6mm_P5.08mm_Horizontal, B.Cu at (177.0, 67.9)
- added R4: 390R, Resistor_THT:R_Axial_DIN0204_L3.6mm_D1.6mm_P5.08mm_Horizontal, B.Cu at (116.0, 91.7)
- added R5: 390R, Resistor_THT:R_Axial_DIN0204_L3.6mm_D1.6mm_P5.08mm_Horizontal, B.Cu at (177.0, 82.4)
- added R6: 390R, Resistor_THT:R_Axial_DIN0204_L3.6mm_D1.6mm_P5.08mm_Horizontal, B.Cu at (177.0, 91.7)
- added R7: 390R, Resistor_THT:R_Axial_DIN0204_L3.6mm_D1.6mm_P5.08mm_Horizontal, B.Cu at (116.0, 96.0)
- added R8: 390R, Resistor_THT:R_Axial_DIN0204_L3.6mm_D1.6mm_P5.08mm_Horizontal, B.Cu at (116.0, 105.3)
- added R9: 390R, Resistor_THT:R_Axial_DIN0204_L3.6mm_D1.6mm_P5.08mm_Horizontal, B.Cu at (177.0, 96.0)
- added SW1: switch_1.00u, 0_west_footprints:SW_Cherry_MX_PCB_1.00u, F.Cu at (127.4, 74.5)
- added SW2: switch_1.00u, 0_west_footprints:SW_Cherry_MX_PCB_1.00u, F.Cu at (146.5, 74.5)
- added SW3: switch_1.00u, 0_west_footprints:SW_Cherry_MX_PCB_1.00u, F.Cu at (165.5, 74.5)
- added SW4: switch_1.00u, 0_west_footprints:SW_Cherry_MX_PCB_1.00u, F.Cu at (127.4, 93.6)
- added SW5: switch_1.00u, 0_west_footprints:SW_Cherry_MX_PCB_1.00u, F.Cu at (146.5, 93.6)
- added SW6: switch_1.00u, 0_west_footprints:SW_Cherry_MX_PCB_1.00u, F.Cu at (165.5, 93.6)
- added SW7: switch_1.00u, 0_west_footprints:SW_Cherry_MX_PCB_1.00u, F.Cu at (127.3, 112.7)
- added SW8: switch_1.00u, 0_west_footprints:SW_Cherry_MX_PCB_1.00u, F.Cu at (146.5, 112.7)
- added SW9: switch_1.00u, 0_west_footprints:SW_Cherry_MX_PCB_1.00u, F.Cu at (165.5, 112.7)
Routing:
- net Net-(D1-K): track 0.00 -> 191.6 mm, vias 0 -> 1
- net Net-(D12-K): track 0.00 -> 91.8 mm, vias 0 -> 2
- net /row_1: track 0.00 -> 86.8 mm, vias 0 -> 1
- net Net-(D11-K): track 0.00 -> 76.7 mm, vias 0 -> 2
- net /row_3: track 0.00 -> 71.9 mm, vias 0 -> 2
- net /collumn_1: track 0.00 -> 69.6 mm, vias 0 -> 1
- net /row_2: track 0.00 -> 64.1 mm, vias 0 -> 1
- net Net-(D5-A): track 0.00 -> 63.1 mm, vias 0 -> 1
- net Net-(D14-K): track 0.00 -> 61.5 mm, vias 0 -> 2
- net Net-(D17-K): track 0.00 -> 60.9 mm, vias 0 -> 3
- net Net-(D10-K): track 0.00 -> 59.4 mm, vias 0 -> 1
- net Net-(D13-K): track 0.00 -> 57.1 mm, vias 0 -> 2
- net /collumn_3: track 0.00 -> 52.1 mm, vias 0 -> 1
- net Net-(D15-K): track 0.00 -> 48.1 mm, vias 0 -> 1
- net Net-(D16-K): track 0.00 -> 47.4 mm, vias 0 -> 2
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- added copper zone on F.Cu, net +5V
- added copper zone on B.Cu, net GND
Other:
- board outline added: 67.6 x 77.6 mm
- copper layers 2 -> 4
- board text added: "Basic Macropad REV1.0"
